File: tamago60/tamago60.kicad_pcb (KiCad board)
At the start: 2 copper layers, 285 x 94.6 mm, 144 parts, among them J1 4105, J2 Cirque FFC, SW1 RESET, SW101 Kailh MX socket, SW102 Kailh MX socket, SW103 Kailh MX socket, SW104 Kailh MX socket, SW105 Kailh MX socket, SW106 Kailh MX socket, SW107 Kailh MX socket, SW108 Kailh MX socket, SW109 Kailh MX socket, SW110 Kailh MX socket, SW111 Kailh MX socket, SW112 Kailh MX socket, SW201 Kailh MX socket, SW202 Kailh MX socket, SW203 Kailh MX socket, SW204 Kailh MX socket, SW205 Kailh MX socket, SW206 Kailh MX socket, SW207 Kailh MX socket, SW208 Kailh MX socket, SW209 Kailh MX socket, SW210 Kailh MX socket, SW211 Kailh MX socket, SW212 Kailh MX socket, SW301 Kailh MX socket, SW302 Kailh MX socket, SW303 Kailh MX socket, SW304 Kailh MX socket, SW305 Kailh MX socket, SW306 Kailh MX socket, SW307 Kailh MX socket, SW308 Kailh MX socket, SW309 Kailh MX socket, SW310 Kailh MX socket, SW311 Kailh MX socket, SW312 Kailh MX socket, SW401 Kailh MX socket, SW402 Kailh MX socket, SW403 Kailh MX socket, SW404 Kailh MX socket, SW405 Kailh MX socket, SW406 Kailh MX socket, SW407 Kailh MX socket, SW408 Kailh MX socket, SW409 Kailh MX socket, SW410 Kailh MX socket, SW411 Kailh MX socket, SW412 Kailh MX socket, SW501 Kailh MX socket, SW502 Kailh MX socket, SW503 Kailh MX socket, SW504 Kailh MX socket, SW505 Kailh MX socket, SW508 Kailh MX socket, SW509 Kailh MX socket, SW510 Kailh MX socket, SW511 Kailh MX socket, SW512 Kailh MX socket, U1 ATmega32U4-A, U2 NCP1117-3.3_SOT223, Y1 16MHz

Commit message: route left side
Parts:
- moved U2 2.41 mm to (203.1, 55.8)
- moved A1 2.00 mm to (210.5, 118.2)
- moved J2 2.00 mm to (200.5, 118.2)
- moved C6 0.40 mm to (201.1, 61.0)
- moved R5 0.40 mm to (205.5, 86.4)
- moved SW1 0.40 mm to (210.5, 86.4)
- turned C1 to 90 degrees
- turned R1 to 180 degrees
Connections:
- C4 pad 1: VBUS -> +3V3
- R1 pad 1: Net-(J1-PadA6) -> Net-(R1-Pad1)
- R2 pad 1: D- -> Net-(R2-Pad1)
- R2 pad 2: Net-(J1-PadA7) -> D-
- R5 pad 2: VBUS -> +3V3
Routing:
- net Col1: track 0.00 -> 222.2 mm, vias 0 -> 8
- net Col2: track 0.00 -> 201.9 mm, vias 0 -> 8
- net Col3: track 0.00 -> 183.3 mm, vias 0 -> 8
- net Col4: track 0.00 -> 164.7 mm, vias 0 -> 8
- net Row5: track 0.00 -> 164.3 mm, vias 0 -> 2
- net VBUS: track 0.00 -> 160.7 mm
- net Col5: track 0.00 -> 149.7 mm, vias 0 -> 8
- net D+: track 0.00 -> 145.4 mm, vias 0 -> 2
- net D-: track 0.00 -> 145.0 mm, vias 0 -> 2
- net Row4: track 0.00 -> 138.1 mm, vias 0 -> 2
- net Row1: track 0.00 -> 137.0 mm, vias 0 -> 2
- net Row2: track 0.00 -> 127.4 mm, vias 0 -> 2
- net Row3: track 0.00 -> 121.0 mm, vias 0 -> 2
- net +3V3: track 0.00 -> 117.6 mm, vias 0 -> 2
- net Col6: track 0.00 -> 107.7 mm, vias 0 -> 7
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- added copper zone on B.Cu, net GND
- added copper zone on F.Cu, net GND

Commit message: rework with rp2040 module
Parts:
- removed C1, C2: 22p, Capacitor_SMD:C_1206_3216Metric
- removed C3, C4: 1u, Capacitor_SMD:C_1206_3216Metric
- removed C5, C6: 10u, Capacitor_SMD:C_1206_3216Metric
- removed the R1 at (200.5, 77.0)
- removed the R2 at (200.5, 79.6)
- removed R5, R6: 5.1k, Resistor_SMD:R_1206_3216Metric
- removed SW1: RESET, Jumper:SolderJumper-2_P1.3mm_Open_Pad1.0x1.5mm
- removed U2: NCP1117-3.3_SOT223, Package_TO_SOT_SMD:SOT-223-3_TabPin2
- removed Y1: 16MHz, Crystal:Crystal_SMD_2520-4Pin_2.5x2.0mm
- added R3: 5.1k, Resistor_SMD:R_1206_3216Metric, B.Cu at (222.3, 89.2)
- added R4: 5.1k, Resistor_SMD:R_1206_3216Metric, B.Cu at (222.3, 91.6)
- U1: value ATmega32U4-A -> kb2040; footprint Package_QFP:TQFP-44_10x10mm_P0.8mm -> kb2040:kb2040; moved to F.Cu
- moved R1 5.22 mm to (79.3, 50.8)
- moved R2 5.22 mm to (76.7, 50.8)
- moved U1 1.00 mm to (210.5, 75.0)
- renumbered R3 to R1, R4 to R2
Connections:
- J2 pad 1: SCK -> unconnected-(J2-Pad1)
- J2 pad 10: unconnected-(J2-Pad10) -> SDA
- J2 pad 2: MISO -> unconnected-(J2-Pad2)
- J2 pad 3: SS -> unconnected-(J2-Pad3)
- J2 pad 5: MOSI -> unconnected-(J2-Pad5)
- J2 pad 9: unconnected-(J2-Pad9) -> SCL
- U1 pad 1: Row1 -> D+
- U1 pad 10: MOSI -> Col5
- U1 pad 11: MISO -> Col6
- U1 pad 12: unconnected-(U1-Pad12) -> Row3
- U1 pad 13: RESET -> Row4
- U1 pad 14: +3V3 -> D-
- U1 pad 15: GND -> VBUS
- U1 pad 16: XTAL2 -> GND
- U1 pad 17: XTAL1 -> unconnected-(U1-Pad17)
- U1 pad 18: Row6 -> +3V3
- U1 pad 19: Row7 -> Row5
- U1 pad 2: VBUS -> Row1
- U1 pad 20: Row8 -> Row6
- U1 pad 21: Row9 -> Row7
- U1 pad 22: Row10 -> Row8
- U1 pad 23: GND -> Row9
- U1 pad 24: +3V3 -> Row10
- U1 pad 25: Col1 -> SCL
- U1 pad 26: Col2 -> SDA
- U1 pad 3: Net-(R2-Pad1) -> Row2
- U1 pad 4: Net-(R1-Pad1) -> GND
- U1 pad 6: Net-(C3-Pad1) -> Col1
- U1 pad 7: VBUS -> Col2
- U1 pad 8: SS -> Col3
- U1 pad 9: SCK -> Col4
Routing:
- net Col1: track 222.2 -> 454.4 mm, vias 8 -> 13
- net Col2: track 201.9 -> 414.4 mm, vias 8 -> 13
- net Col3: track 183.3 -> 377.6 mm, vias 8 -> 13
- net Col4: track 164.7 -> 339.5 mm, vias 8 -> 13
- net Col5: track 149.7 -> 316.7 mm, vias 8 -> 13
- net Col6: track 107.7 -> 225.3 mm, vias 7 -> 11
- net MOSI: track 68.6 -> 0.00 mm, vias 2 -> 0
- net SS: track 67.5 -> 0.00 mm, vias 2 -> 0
- net MISO: track 58.9 -> 0.00 mm, vias 2 -> 0
- net SCK: track 57.1 -> 0.00 mm, vias 2 -> 0
- net Row10: track 101.4 -> 150.9 mm, vias 0 -> 1
- net +3V3: track 117.6 -> 68.3 mm, vias 2 -> 0
- net SCL: track 0.00 -> 46.5 mm
- net SDA: track 0.00 -> 44.8 mm
- net Row9: track 95.2 -> 130.3 mm, vias 0 -> 1
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Other:
- board text added: "Tamago v2 August 2023 EggsWorks, LLC github.com/eggsworks www.eggs.works"

Commit message: mfgr prep
Parts:
- added XSW101: Kailh MX socket, tamago60:Kailh_socket_MX, B.Cu at (83.5, 58.2)
- added XSW102: Kailh MX socket, tamago60:Kailh_socket_MX, B.Cu at (102.5, 58.2)
- added XSW103: Kailh MX socket, tamago60:Kailh_socket_MX, B.Cu at (121.5, 58.2)
- added XSW104: Kailh MX socket, tamago60:Kailh_socket_MX, B.Cu at (140.6, 58.2)
- added XSW105: Kailh MX socket, tamago60:Kailh_socket_MX, B.Cu at (159.6, 58.2)
- added XSW106: Kailh MX socket, tamago60:Kailh_socket_MX, B.Cu at (178.7, 58.2)
- added XSW107: Kailh MX socket, tamago60:Kailh_socket_MX, B.Cu at (243.6, 58.2)
- added XSW108: Kailh MX socket, tamago60:Kailh_socket_MX, B.Cu at (262.7, 58.2)
- added XSW109: Kailh MX socket, tamago60:Kailh_socket_MX, B.Cu at (281.7, 58.2)
- added XSW110: Kailh MX socket, tamago60:Kailh_socket_MX, B.Cu at (300.8, 58.2)
- added XSW111: Kailh MX socket, tamago60:Kailh_socket_MX, B.Cu at (319.8, 58.2)
- added XSW112: Kailh MX socket, tamago60:Kailh_socket_MX, B.Cu at (338.9, 58.2)
- added XSW201: Kailh MX socket, tamago60:Kailh_socket_MX, B.Cu at (82.2, 69.6)
- added XSW202: Kailh MX socket, tamago60:Kailh_socket_MX, B.Cu at (102.5, 77.2)
- added XSW203: Kailh MX socket, tamago60:Kailh_socket_MX, B.Cu at (121.5, 77.2)
- added XSW204: Kailh MX socket, tamago60:Kailh_socket_MX, B.Cu at (140.6, 77.2)
- added XSW205: Kailh MX socket, tamago60:Kailh_socket_MX, B.Cu at (159.6, 77.2)
- added XSW206: Kailh MX socket, tamago60:Kailh_socket_MX, B.Cu at (178.7, 77.2)
- added XSW207: Kailh MX socket, tamago60:Kailh_socket_MX, B.Cu at (243.6, 77.2)
- added XSW208: Kailh MX socket, tamago60:Kailh_socket_MX, B.Cu at (262.7, 77.2)
- added XSW209: Kailh MX socket, tamago60:Kailh_socket_MX, B.Cu at (281.7, 77.2)
- added XSW210: Kailh MX socket, tamago60:Kailh_socket_MX, B.Cu at (300.8, 77.2)
- added XSW211: Kailh MX socket, tamago60:Kailh_socket_MX, B.Cu at (318.5, 69.6)
- added XSW212: Kailh MX socket, tamago60:Kailh_socket_MX, B.Cu at (338.9, 77.2)
- added XSW301: Kailh MX socket, tamago60:Kailh_socket_MX, B.Cu at (83.5, 96.3)
- added XSW302: Kailh MX socket, tamago60:Kailh_socket_MX, B.Cu at (102.5, 96.3)
- added XSW303: Kailh MX socket, tamago60:Kailh_socket_MX, B.Cu at (121.5, 96.3)
- added XSW304: Kailh MX socket, tamago60:Kailh_socket_MX, B.Cu at (140.6, 96.3)
- added XSW305: Kailh MX socket, tamago60:Kailh_socket_MX, B.Cu at (159.6, 96.3)
- added XSW306: Kailh MX socket, tamago60:Kailh_socket_MX, B.Cu at (178.7, 96.3)
- added XSW307: Kailh MX socket, tamago60:Kailh_socket_MX, B.Cu at (243.6, 96.3)
- added XSW308: Kailh MX socket, tamago60:Kailh_socket_MX, B.Cu at (262.7, 96.3)
- added XSW309: Kailh MX socket, tamago60:Kailh_socket_MX, B.Cu at (281.7, 96.3)
- added XSW310: Kailh MX socket, tamago60:Kailh_socket_MX, B.Cu at (300.8, 96.3)
- added XSW311: Kailh MX socket, tamago60:Kailh_socket_MX, B.Cu at (319.8, 96.3)
- added XSW312: Kailh MX socket, tamago60:Kailh_socket_MX, B.Cu at (338.9, 96.3)
- added XSW401: Kailh MX socket, tamago60:Kailh_socket_MX, B.Cu at (83.5, 115.3)
- added XSW402: Kailh MX socket, tamago60:Kailh_socket_MX, B.Cu at (102.5, 115.3)
- added XSW403: Kailh MX socket, tamago60:Kailh_socket_MX, B.Cu at (121.5, 115.3)
- added XSW404: Kailh MX socket, tamago60:Kailh_socket_MX, B.Cu at (140.6, 115.3)
- added XSW405: Kailh MX socket, tamago60:Kailh_socket_MX, B.Cu at (159.6, 115.3)
- added XSW406: Kailh MX socket, tamago60:Kailh_socket_MX, B.Cu at (178.7, 115.3)
- added XSW407: Kailh MX socket, tamago60:Kailh_socket_MX, B.Cu at (243.6, 115.3)
- added XSW408: Kailh MX socket, tamago60:Kailh_socket_MX, B.Cu at (262.7, 115.3)
- added XSW409: Kailh MX socket, tamago60:Kailh_socket_MX, B.Cu at (281.7, 115.3)
- added XSW410: Kailh MX socket, tamago60:Kailh_socket_MX, B.Cu at (300.8, 115.3)
- added XSW411: Kailh MX socket, tamago60:Kailh_socket_MX, B.Cu at (319.8, 115.3)
- added XSW412: Kailh MX socket, tamago60:Kailh_socket_MX, B.Cu at (338.9, 115.3)
- added XSW501: Kailh MX socket, tamago60:Kailh_socket_MX, B.Cu at (83.5, 134.4)
- added XSW502: Kailh MX socket, tamago60:Kailh_socket_MX, B.Cu at (102.5, 134.4)
- added XSW503: Kailh MX socket, tamago60:Kailh_socket_MX, B.Cu at (121.5, 134.4)
- added XSW504: Kailh MX socket, tamago60:Kailh_socket_MX, B.Cu at (140.6, 134.4)
- added XSW505: Kailh MX socket, tamago60:Kailh_socket_MX, B.Cu at (169.2, 134.4)
- added XSW508: Kailh MX socket, tamago60:Kailh_socket_MX, B.Cu at (251.8, 126.8)
- added XSW509: Kailh MX socket, tamago60:Kailh_socket_MX, B.Cu at (281.7, 134.4)
- added XSW510: Kailh MX socket, tamago60:Kailh_socket_MX, B.Cu at (300.8, 134.4)
- added XSW511: Kailh MX socket, tamago60:Kailh_socket_MX, B.Cu at (319.8, 134.4)
- added XSW512: Kailh MX socket, tamago60:Kailh_socket_MX, B.Cu at (338.9, 134.4)
- SW101, SW102, SW103, SW104, SW105, SW106, SW107, SW108, SW109, SW110, SW111, SW112, SW201, SW202, SW203, SW204, SW205, SW206, SW207, SW208, SW209, SW210, SW211, SW212, SW301, SW302, SW303, SW304, SW305, SW306, SW307, SW308, SW309, SW310, SW311, SW312, SW401, SW402, SW403, SW404, SW405, SW406, SW407, SW408, SW409, SW410, SW411, SW412, SW501, SW502, SW503, SW504, SW505, SW508, SW509, SW510, SW511, SW512: footprint tamago60:Kailh_socket_MX_platemount -> tamago60:Kailh_socket_MX_position

Commit message: fixes for production
Routing:
- net Col5: track 316.7 -> 341.0 mm
- net Col2: track 414.2 -> 436.9 mm
- net Col4: track 339.5 -> 362.1 mm
- net Col3: track 377.6 -> 399.7 mm
- net Col6: track 225.0 -> 242.4 mm
- net +3V3: track 68.3 -> 71.1 mm
- net Col1: track 454.4 -> 454.3 mm, vias 13 -> 1

Commit message: layout with choc sockets
Parts:
- removed D101: 1N1418, Diode_SMD:D_SOD-123
- removed MH2, MH4, MH5: MountingHole, tamago60:circle_mounting_hole
- removed REF** (x2): Stabilizer_Cherry_MX_2.00u, tamago60:Stabilizer_Cherry_MX_2.00u
- removed U1: kb2040, kb2040:kb2040
- SW101, SW102, SW103, SW104, SW105, SW106, SW107, SW108, SW109, SW110, SW111, SW112, SW201, SW202, SW203, SW204, SW205, SW206, SW207, SW208, SW209, SW210, SW211, SW212, SW301, SW302, SW303, SW304, SW305, SW306, SW307, SW308, SW309, SW310, SW311, SW312, SW401, SW402, SW403, SW404, SW405, SW406, SW407, SW408, SW409, SW410, SW411, SW412, SW501, SW502, SW503, SW504, SW505, SW508, SW509, SW510, SW511, SW512: footprint tamago60:Kailh_socket_MX_position -> tamago60:Kailh_socket_PG1350_position
- XSW101, XSW102, XSW103, XSW104, XSW105, XSW106, XSW107, XSW108, XSW109, XSW110, XSW111, XSW112, XSW201, XSW202, XSW203, XSW204, XSW205, XSW206, XSW207, XSW208, XSW209, XSW210, XSW211, XSW212, XSW301, XSW302, XSW303, XSW304, XSW305, XSW306, XSW307, XSW308, XSW309, XSW310, XSW311, XSW312, XSW401, XSW402, XSW403, XSW404, XSW405, XSW406, XSW407, XSW408, XSW409, XSW410, XSW411, XSW412, XSW501, XSW502, XSW503, XSW504, XSW505, XSW508, XSW509, XSW510, XSW511, XSW512: footprint tamago60:Kailh_socket_MX -> tamago60:Kailh_socket_PG1350; moved to F.Cu
- moved J2 21.2 mm to (220.5, 111.3), turned to 90 degrees
- moved R2 20.3 mm to (97.0, 51.0), turned to -90 degrees
- moved R1 15.1 mm to (94.4, 51.0), turned to -90 degrees
- moved XSW106 14.1 mm to (165.8, 63.8), turned to 180 degrees
- moved XSW206 13.4 mm to (165.8, 80.8), turned to 180 degrees
- moved XSW105 13.2 mm to (147.7, 63.8), turned to 180 degrees
- moved XSW306 13.0 mm to (165.8, 97.8), turned to 180 degrees
- moved XSW406 13.0 mm to (165.8, 114.9), turned to 180 degrees
- moved XSW505 12.7 mm to (156.7, 131.9), turned to 180 degrees
- moved XSW501 12.5 mm to (80.5, 122.2)
- moved XSW205 12.5 mm to (147.7, 80.8), turned to 180 degrees
- moved XSW104 12.3 mm to (129.7, 63.8), turned to 180 degrees
- moved XSW305 12.1 mm to (147.7, 97.8), turned to 180 degrees
- moved XSW405 12.0 mm to (147.7, 114.9), turned to 180 degrees
- moved XSW211 11.9 mm to (322.5, 80.8)
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Connections:
- XSW101 pad 1: Net-(D101-Pad2) -> Col1
- XSW101 pad 2: Col1 -> Net-(D201-Pad2)
Routing:
- net Col1: track 454.3 -> 0.00 mm, vias 1 -> 0
- net Col2: track 436.9 -> 0.00 mm, vias 13 -> 0
- net Col3: track 399.7 -> 0.00 mm, vias 13 -> 0
- net Col4: track 362.1 -> 0.00 mm, vias 13 -> 0
- net Col5: track 341.0 -> 0.00 mm, vias 13 -> 0
- net Col6: track 242.4 -> 0.00 mm, vias 11 -> 0
- net Row5: track 160.2 -> 0.00 mm
- net Row10: track 150.9 -> 0.00 mm, vias 1 -> 0
- net VBUS: track 147.2 -> 0.00 mm
- net D-: track 141.5 -> 0.00 mm, vias 1 -> 0
- net D+: track 140.5 -> 0.00 mm, vias 1 -> 0
- net Row9: track 130.3 -> 0.00 mm, vias 1 -> 0
- net Row6: track 130.1 -> 0.00 mm, vias 1 -> 0
- net Row4: track 118.4 -> 0.00 mm
- net Row7: track 117.1 -> 0.00 mm, vias 1 -> 0
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