File: tamago60/tamago60.kicad_pcb (KiCad board)
At the start: 2 copper layers, 285 x 94.6 mm, 184 parts, among them J1 4105, J2 Cirque FFC, SW101 Kailh MX socket, SW102 Kailh MX socket, SW103 Kailh MX socket, SW104 Kailh MX socket, SW105 Kailh MX socket, SW106 Kailh MX socket, SW107 Kailh MX socket, SW108 Kailh MX socket, SW109 Kailh MX socket, SW110 Kailh MX socket, SW111 Kailh MX socket, SW112 Kailh MX socket, SW201 Kailh MX socket, SW202 Kailh MX socket, SW203 Kailh MX socket, SW204 Kailh MX socket, SW205 Kailh MX socket, SW206 Kailh MX socket, SW207 Kailh MX socket, SW208 Kailh MX socket, SW209 Kailh MX socket, SW210 Kailh MX socket, SW211 Kailh MX socket, SW212 Kailh MX socket, SW301 Kailh MX socket, SW302 Kailh MX socket, SW303 Kailh MX socket, SW304 Kailh MX socket, SW305 Kailh MX socket, SW306 Kailh MX socket, SW307 Kailh MX socket, SW308 Kailh MX socket, SW309 Kailh MX socket, SW310 Kailh MX socket, SW311 Kailh MX socket, SW312 Kailh MX socket, SW401 Kailh MX socket, SW402 Kailh MX socket, SW403 Kailh MX socket, SW404 Kailh MX socket, SW405 Kailh MX socket, SW406 Kailh MX socket, SW407 Kailh MX socket, SW408 Kailh MX socket, SW409 Kailh MX socket, SW410 Kailh MX socket, SW411 Kailh MX socket, SW412 Kailh MX socket, SW501 Kailh MX socket, SW502 Kailh MX socket, SW503 Kailh MX socket, SW504 Kailh MX socket, SW505 Kailh MX socket, SW508 Kailh MX socket, SW509 Kailh MX socket, SW510 Kailh MX socket, SW511 Kailh MX socket, SW512 Kailh MX socket

Commit message: routing
Parts:
- added D101: 1N1418, Diode_SMD:D_SOD-123, B.Cu at (70.5, 64.2)
- added D506: 1N1418, Diode_SMD:D_SOD-123, B.Cu at (192.4, 134.8)
- added D507: 1N1418, Diode_SMD:D_SOD-123, B.Cu at (228.6, 134.7)
- added SW506: ~, tamago60:SW_D2F-FL, F.Cu at (201.5, 134.7)
- added SW507: ~, tamago60:SW_D2F-FL, F.Cu at (219.5, 134.7)
- added U1: kb2040, kb2040:kb2040, F.Cu at (210.5, 65.3)
- XSW101, XSW102, XSW103, XSW104, XSW105, XSW106, XSW107, XSW108, XSW109, XSW110, XSW111, XSW112, XSW201, XSW202, XSW203, XSW204, XSW205, XSW206, XSW207, XSW208, XSW209, XSW210, XSW211, XSW212, XSW301, XSW302, XSW303, XSW304, XSW305, XSW306, XSW307, XSW308, XSW309, XSW310, XSW311, XSW312, XSW401, XSW402, XSW403, XSW404, XSW405, XSW406, XSW407, XSW408, XSW409, XSW410, XSW411, XSW412, XSW501, XSW502, XSW503, XSW504, XSW505, XSW508, XSW509, XSW510, XSW511, XSW512: value Kailh MX socket -> Kailh choc socket
- moved D201 20.8 mm to (70.5, 81.2), turned to 90 degrees
- moved D301 20.7 mm to (70.5, 97.1), turned to 90 degrees
- moved D401 20.1 mm to (70.5, 118.3), turned to 90 degrees
- moved D302 19.6 mm to (88.5, 101.9), turned to 90 degrees
- moved D402 19.3 mm to (88.5, 118.3), turned to 90 degrees
- moved D501 19.2 mm to (70.5, 133.2), turned to 90 degrees
- moved XSW401 10.9 mm to (75.5, 114.9), turned to 180 degrees
- moved XSW312 10.9 mm to (345.5, 88.2)
- moved D102 10.8 mm to (103.5, 66.8), turned to 90 degrees
- moved D202 10.8 mm to (103.5, 84.3), turned to 90 degrees
- moved D505 8.78 mm to (170.0, 124.0)
- moved D508 8.77 mm to (251.0, 123.7)
- moved #LOGO1 3.75 mm to (210.5, 58.9)
- turned SW312 to 180 degrees
- turned SW401 to 0 degrees
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- renumbered MH3 to MH2, MH6 to MH3
Connections:
- D201 pad 2: Net-(D201-Pad2) -> Net-(D201-A)
- XSW101 pad 1: Col1 -> Net-(D101-A)
- XSW101 pad 2: Net-(D201-Pad2) -> Col1
- XSW201 pad 2: Net-(D201-Pad2) -> Net-(D201-A)
Routing:
- net Col1: track 0.00 -> 453.5 mm
- net Col2: track 0.00 -> 443.5 mm
- net Col3: track 0.00 -> 402.8 mm
- net Col4: track 0.00 -> 377.9 mm
- net Col6: track 0.00 -> 337.1 mm
- net Col5: track 0.00 -> 326.4 mm
- net Row5: track 0.00 -> 222.8 mm, vias 0 -> 4
- net Row4: track 0.00 -> 176.6 mm, vias 0 -> 5
- net Row2: track 0.00 -> 161.6 mm, vias 0 -> 6
- net Row3: track 0.00 -> 155.6 mm, vias 0 -> 6
- net VBUS: track 0.00 -> 154.8 mm, vias 0 -> 1
- net Row1: track 0.00 -> 153.7 mm, vias 0 -> 6
- net Row10: track 0.00 -> 148.1 mm, vias 0 -> 5
- net Row9: track 0.00 -> 141.4 mm, vias 0 -> 6
- net D-: track 0.00 -> 139.2 mm, vias 0 -> 1
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Other:
- board text added: "Tamago III December 2023 EggsWorks, LLC github.com/eggsworks www.eggs.works"
- board text removed: "Tamago v2 August 2023 EggsWorks, LLC github.com/eggsworks www.eggs.works"
