File: tamago60/tamago60.kicad_sch (KiCad schematic)
At the start: 6 parts

Commit message: routing
Parts:
- removed MH2, MH4, MH5: MountingHole, tamago60:circle_mounting_hole, symbol Mechanical:MountingHole
- renumbered MH3 to MH2, MH6 to MH3
Other:
- moved on the sheet: MH1, MH2, MH3
