File: tamago60/tamago60_matrix.kicad_sch (KiCad schematic)
At the start: 63 parts, among them SW101 switch_with_diode, SW102 switch_with_diode, SW103 switch_with_diode, SW104 switch_with_diode, SW105 switch_with_diode, SW106 switch_with_diode, SW107 switch_with_diode, SW108 switch_with_diode, SW109 switch_with_diode, SW110 switch_with_diode, SW111 switch_with_diode, SW112 switch_with_diode, SW201 switch_with_diode, SW202 switch_with_diode, SW203 switch_with_diode, SW204 switch_with_diode, SW205 switch_with_diode, SW206 switch_with_diode, SW207 switch_with_diode, SW208 switch_with_diode, SW209 switch_with_diode, SW210 switch_with_diode, SW211 switch_with_diode, SW212 switch_with_diode, SW301 switch_with_diode, SW302 switch_with_diode, SW303 switch_with_diode, SW304 switch_with_diode, SW305 switch_with_diode, SW306 switch_with_diode, SW307 switch_with_diode, SW308 switch_with_diode, SW309 switch_with_diode, SW310 switch_with_diode, SW311 switch_with_diode, SW312 switch_with_diode, SW401 switch_with_diode, SW402 switch_with_diode, SW403 switch_with_diode, SW404 switch_with_diode, SW405 switch_with_diode, SW406 switch_with_diode, SW407 switch_with_diode, SW408 switch_with_diode, SW409 switch_with_diode, SW410 switch_with_diode, SW411 switch_with_diode, SW412 switch_with_diode, SW501 switch_with_diode, SW502 switch_with_diode, SW503 switch_with_diode, SW504 switch_with_diode, SW505 switch_with_diode, SW506 switch_with_diode, SW507 switch_with_diode, SW508 switch_with_diode, SW509 switch_with_diode, SW510 switch_with_diode, SW511 switch_with_diode, SW512 switch_with_diode, SW600 JP19

Commit message: Finalize v1 design
Other:
- company: (none) -> EggsWorks, LLC
- title: (none) -> tamago60
Changed lines of the file:
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@@
 (kicad_sch (version 20211123) (generator eeschema)
   (paper "A4")
+  (title_block
+    (title "tamago60")
+    (date "2023-04-13")
+    (rev "v1")
+    (company "EggsWorks, LLC")
+  )
   (junction (at 104.775 100.965) (diameter 0) (color 0 0 0 0)
   )

Commit message: Fix 2u position defect - bump to v1.1
Parts:
- SW505: footprint tamago60:Choc_Hotswap_2u -> tamago60:Choc_Hotswap_2u_left
Changed lines of the file:
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@@
       (effects (font (size 1.27 1.27)) (justify left) hide)
     )
-    (property "Footprint" "tamago60:Choc_Hotswap_2u" (id 2) (at 108.585 136.525 0)
+    (property "Footprint" "tamago60:Choc_Hotswap_2u_left" (id 2) (at 108.585 136.525 0)
       (effects (font (size 1.27 1.27)) hide)
     )
@@
       (effects (font (size 1.27 1.27)) hide)
     )
-    (property "Footprint" "tamago60:Choc_Hotswap_2u" (id 2) (at 98.425 127.635 0)
-      (effects (font (size 1.27 1.27)) hide)
-    )
+    (property "Footprint" "tamago60:Choc_Hotswap_2u_left" (id 2) (at 98.425 127.635 0)
+      (effects (font (size 1.27 1.27)) hide)
+    )

Commit message: Replace JST with 2mm, move its position; update schematic to be consistent with PCB
Parts:
- SW508: footprint tamago60:Choc_Hotswap_2u -> tamago60:Choc_Hotswap_2u_right
Changed lines of the file:
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@@
       (effects (font (size 1.27 1.27)) (justify left) hide)
     )
-    (property "Footprint" "tamago60:Choc_Hotswap_2u" (id 2) (at 220.345 136.525 0)
+    (property "Footprint" "tamago60:Choc_Hotswap_2u_right" (id 2) (at 220.345 136.525 0)
       (effects (font (size 1.27 1.27)) hide)
     )
@@
       (effects (font (size 1.27 1.27)) hide)
     )
-    (property "Footprint" "tamago60:Choc_Hotswap_2u" (id 2) (at 210.185 127.635 0)
-      (effects (font (size 1.27 1.27)) hide)
-    )
+    (property "Footprint" "tamago60:Choc_Hotswap_2u_right" (id 2) (at 210.185 127.635 0)
+      (effects (font (size 1.27 1.27)) hide)
+    )

Commit message: Initial layout for tamago v2
Parts:
- removed D600: D, Diode_SMD:D_SOD-123, symbol Device:D
- removed JP1: SolderJumper_3_Open, Jumper:SolderJumper-3_P1.3mm_Open_Pad1.0x1.5mm_NumberLabels, symbol Jumper:SolderJumper_3_Open
- removed unit 2 of SW101
- removed unit 2 of SW102
- removed unit 2 of SW103
- removed unit 2 of SW104
- removed unit 2 of SW105
- removed unit 2 of SW106
- removed unit 2 of SW107
- removed unit 2 of SW108
- removed unit 2 of SW109
- removed unit 2 of SW110
- removed unit 2 of SW111
- removed unit 2 of SW112
- removed unit 2 of SW201
- removed unit 2 of SW202
- removed unit 2 of SW203
- removed unit 2 of SW204
- removed unit 2 of SW205
- removed unit 2 of SW206
- removed unit 2 of SW207
- removed unit 2 of SW208
- removed unit 2 of SW209
- removed unit 2 of SW210
- removed unit 2 of SW211
- removed unit 2 of SW212
- removed unit 2 of SW301
- removed unit 2 of SW302
- removed unit 2 of SW303
- removed unit 2 of SW304
- removed unit 2 of SW305
- removed unit 2 of SW306
- removed unit 2 of SW307
- removed unit 2 of SW308
- removed unit 2 of SW309
- removed unit 2 of SW310
- removed unit 2 of SW311
- removed unit 2 of SW312
- removed unit 2 of SW401
- removed unit 2 of SW402
- removed unit 2 of SW403
- removed unit 2 of SW404
- removed unit 2 of SW405
- removed unit 2 of SW406
- removed unit 2 of SW407
- removed unit 2 of SW408
- removed unit 2 of SW409
- removed unit 2 of SW410
- removed unit 2 of SW411
- removed unit 2 of SW412
- removed unit 2 of SW501
- removed unit 2 of SW502
- removed unit 2 of SW503
- removed unit 2 of SW504
- removed unit 2 of SW505
- removed SW506, SW507: switch_with_diode, tamago60:Choc_Hotswap, symbol tamago60:switch_with_diode
- removed unit 2 of SW508
- removed unit 2 of SW509
- removed unit 2 of SW510
- removed unit 2 of SW511
- removed unit 2 of SW512
- removed SW600: JP19, tamago60:JP19, symbol tamago60:JP19
- added D101, D102, D103, D104, D105, D106, D107, D108, D109, D110, D111, D112, D201, D202, D203, D204, D205, D206, D207, D208, D209, D210, D211, D212, D301, D302, D303, D304, D305, D306, D307, D308, D309, D310, D311, D312, D401, D402, D403, D404, D405, D406, D407, D408, D409, D410, D411, D412, D501, D502, D503, D504, D505, D508, D509, D510, D511, D512: 1N1418, Diode_SMD:D_SOD-123, symbol Device:D_Small_Filled
- SW101, SW102, SW103, SW104, SW105, SW106, SW202, SW203, SW204, SW205, SW206, SW211, SW301, SW302, SW303, SW304, SW305, SW306, SW401, SW402, SW403, SW404, SW405, SW406, SW501, SW502, SW503, SW504: value switch_with_diode -> Kailh MX socket; footprint tamago60:Choc_Hotswap -> tamago60:Kailh_socket_MX_platemount; symbol tamago60:switch_with_diode -> tamago60:SW_Push_flipped
- SW107, SW108, SW109, SW110, SW111, SW112, SW201, SW207, SW208, SW209, SW210, SW212, SW307, SW308, SW309, SW310, SW311, SW312, SW407, SW408, SW409, SW410, SW411, SW412, SW509, SW510, SW511, SW512: value switch_with_diode -> Kailh MX socket; footprint tamago60:Choc_Hotswap -> tamago60:Kailh_socket_MX_platemount; symbol tamago60:switch_with_diode -> Switch:SW_Push
- SW505: value switch_with_diode -> Kailh MX socket; footprint tamago60:Choc_Hotswap_2u_left -> tamago60:Kailh_socket_MX_platemount; symbol tamago60:switch_with_diode -> tamago60:SW_Push_flipped
- SW508: value switch_with_diode -> Kailh MX socket; footprint tamago60:Choc_Hotswap_2u_right -> tamago60:Kailh_socket_MX_platemount; symbol tamago60:switch_with_diode -> Switch:SW_Push
Connections:
- net Col1: now also SW101.2, SW301.2, SW401.2, SW501.2; no longer SW101.1 (SW), SW301.1 (SW), SW401.1 (SW), SW501.1 (SW)
- net Col2: now also SW102.2, SW202.2, SW211.2, SW302.2, SW402.2, SW502.2; no longer SW102.1 (SW), SW202.1 (SW), SW211.1 (SW), SW302.1 (SW), SW402.1 (SW), SW502.1 (SW)
- net Col3: now also SW103.2, SW203.2, SW303.2, SW403.2, SW503.2; no longer SW103.1 (SW), SW203.1 (SW), SW303.1 (SW), SW403.1 (SW), SW503.1 (SW)
- net Col4: now also SW104.2, SW204.2, SW304.2, SW404.2, SW504.2; no longer SW104.1 (SW), SW204.1 (SW), SW304.1 (SW), SW404.1 (SW), SW504.1 (SW)
- net Col5: now also SW105.2, SW205.2, SW305.2, SW405.2, SW505.2; no longer SW105.1 (SW), SW205.1 (SW), SW305.1 (SW), SW405.1 (SW), SW505.1 (SW)
- net Col6: now also SW106.2, SW206.2, SW306.2, SW406.2; no longer SW106.1 (SW), SW206.1 (SW), SW306.1 (SW), SW406.1 (SW)
- net Row1: now also D101.1 (K), D102.1 (K), D103.1 (K), D104.1 (K), D105.1 (K), D106.1 (K)
- net Row10: now also D508.1 (K), D509.1 (K), D510.1 (K), D511.1 (K), D512.1 (K)
- net Row2: now also D201.1 (K), D202.1 (K), D203.1 (K), D204.1 (K), D205.1 (K), D206.1 (K)
- net Row3: now also D301.1 (K), D302.1 (K), D303.1 (K), D304.1 (K), D305.1 (K), D306.1 (K)
- net Row4: now also D401.1 (K), D402.1 (K), D403.1 (K), D404.1 (K), D405.1 (K), D406.1 (K)
- net Row5: now also D501.1 (K), D502.1 (K), D503.1 (K), D504.1 (K), D505.1 (K)
- net Row6: now also D107.1 (K), D108.1 (K), D109.1 (K), D110.1 (K), D111.1 (K), D112.1 (K)
- net Row7: now also D207.1 (K), D208.1 (K), D209.1 (K), D210.1 (K), D211.1 (K), D212.1 (K)
- net Row8: now also D307.1 (K), D308.1 (K), D309.1 (K), D310.1 (K), D311.1 (K), D312.1 (K)
- net Row9: now also D407.1 (K), D408.1 (K), D409.1 (K), D410.1 (K), D411.1 (K), D412.1 (K)
- net at SW209.2: now also D209.2 (A)
- net at SW408.2: now also D408.2 (A)
- net at SW411.2: now also D411.2 (A)
- net at SW212.2: now also D212.2 (A)
- net at SW309.2: now also D309.2 (A)
- net at SW310.2: now also D310.2 (A)
- net at SW412.2: now also D412.2 (A)
- net at SW107.2: now also D107.2 (A)
- net at SW409.2: now also D409.2 (A)
- net at SW111.2: now also D111.2 (A)
- net at SW509.2: now also D509.2 (A)
- net at SW407.2: now also D407.2 (A)
- net at SW410.2: now also D410.2 (A)
- net at SW508.2: now also D508.2 (A)
- net at SW510.2: now also D510.2 (A)
- net at SW112.2: now also D112.2 (A)
- net at SW210.2: now also D210.2 (A)
- net at SW307.2: now also D307.2 (A)
- net at SW108.2: now also D108.2 (A)
- net at SW312.2: now also D312.2 (A)
- net at SW201.2: now also D201.2 (A)
- net at SW308.2: now also D308.2 (A)
- net at SW511.2: now also D511.2 (A)
- net at SW208.2: now also D208.2 (A)
- net at SW311.2: now also D311.2 (A)
- net at SW512.2: now also D512.2 (A)
- net at SW109.2: now also D109.2 (A)
- net at SW207.2: now also D207.2 (A)
- net at SW110.2: now also D110.2 (A)
- new net: D102.2 (A), SW102.1
- new net: D305.2 (A), SW305.1
- new net: D204.2 (A), SW204.1
- new net: D206.2 (A), SW206.1
- new net: D203.2 (A), SW203.1
- new net: D401.2 (A), SW401.1
- new net: D106.2 (A), SW106.1
- new net: D103.2 (A), SW103.1
- new net: D501.2 (A), SW501.1
- new net: D402.2 (A), SW402.1
- new net: D406.2 (A), SW406.1
- new net: D404.2 (A), SW404.1
- new net: D405.2 (A), SW405.1
- new net: D502.2 (A), SW502.1
- new net: D301.2 (A), SW301.1
- new net: D101.2 (A), SW101.1
- new net: D104.2 (A), SW104.1
- new net: D303.2 (A), SW303.1
- new net: D105.2 (A), SW105.1
- new net: D504.2 (A), SW504.1
- new net: D202.2 (A), SW202.1
- new net: D211.2 (A), SW211.1
- new net: D306.2 (A), SW306.1
- new net: D302.2 (A), SW302.1
- new net: D505.2 (A), SW505.1
- new net: D205.2 (A), SW205.1
- new net: D403.2 (A), SW403.1
- new net: D503.2 (A), SW503.1
- new net: D304.2 (A), SW304.1
Other:
- moved on the sheet: SW101, SW102, SW103, SW104, SW105, SW106, SW202, SW203, SW204, SW205, SW206, SW211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

Commit message: mfgr prep
Parts:
- XSW101: renamed from SW101; footprint tamago60:Kailh_socket_MX_platemount -> tamago60:Kailh_socket_MX
- XSW102: renamed from SW102; footprint tamago60:Kailh_socket_MX_platemount -> tamago60:Kailh_socket_MX
- XSW103: renamed from SW103; footprint tamago60:Kailh_socket_MX_platemount -> tamago60:Kailh_socket_MX
- XSW104: renamed from SW104; footprint tamago60:Kailh_socket_MX_platemount -> tamago60:Kailh_socket_MX
- XSW105: renamed from SW105; footprint tamago60:Kailh_socket_MX_platemount -> tamago60:Kailh_socket_MX
- XSW106: renamed from SW106; footprint tamago60:Kailh_socket_MX_platemount -> tamago60:Kailh_socket_MX
- XSW107: renamed from SW107; footprint tamago60:Kailh_socket_MX_platemount -> tamago60:Kailh_socket_MX
- XSW108: renamed from SW108; footprint tamago60:Kailh_socket_MX_platemount -> tamago60:Kailh_socket_MX
- XSW109: renamed from SW109; footprint tamago60:Kailh_socket_MX_platemount -> tamago60:Kailh_socket_MX
- XSW110: renamed from SW110; footprint tamago60:Kailh_socket_MX_platemount -> tamago60:Kailh_socket_MX
- XSW111: renamed from SW111; footprint tamago60:Kailh_socket_MX_platemount -> tamago60:Kailh_socket_MX
- XSW112: renamed from SW112; footprint tamago60:Kailh_socket_MX_platemount -> tamago60:Kailh_socket_MX
- XSW201: renamed from SW201; footprint tamago60:Kailh_socket_MX_platemount -> tamago60:Kailh_socket_MX
- XSW202: renamed from SW202; footprint tamago60:Kailh_socket_MX_platemount -> tamago60:Kailh_socket_MX
- XSW203: renamed from SW203; footprint tamago60:Kailh_socket_MX_platemount -> tamago60:Kailh_socket_MX
- XSW204: renamed from SW204; footprint tamago60:Kailh_socket_MX_platemount -> tamago60:Kailh_socket_MX
- XSW205: renamed from SW205; footprint tamago60:Kailh_socket_MX_platemount -> tamago60:Kailh_socket_MX
- XSW206: renamed from SW206; footprint tamago60:Kailh_socket_MX_platemount -> tamago60:Kailh_socket_MX
- XSW207: renamed from SW207; footprint tamago60:Kailh_socket_MX_platemount -> tamago60:Kailh_socket_MX
- XSW208: renamed from SW208; footprint tamago60:Kailh_socket_MX_platemount -> tamago60:Kailh_socket_MX
- XSW209: renamed from SW209; footprint tamago60:Kailh_socket_MX_platemount -> tamago60:Kailh_socket_MX
- XSW210: renamed from SW210; footprint tamago60:Kailh_socket_MX_platemount -> tamago60:Kailh_socket_MX
- XSW211: renamed from SW211; footprint tamago60:Kailh_socket_MX_platemount -> tamago60:Kailh_socket_MX
- XSW212: renamed from SW212; footprint tamago60:Kailh_socket_MX_platemount -> tamago60:Kailh_socket_MX
- XSW301: renamed from SW301; footprint tamago60:Kailh_socket_MX_platemount -> tamago60:Kailh_socket_MX
- XSW302: renamed from SW302; footprint tamago60:Kailh_socket_MX_platemount -> tamago60:Kailh_socket_MX
- XSW303: renamed from SW303; footprint tamago60:Kailh_socket_MX_platemount -> tamago60:Kailh_socket_MX
- XSW304: renamed from SW304; footprint tamago60:Kailh_socket_MX_platemount -> tamago60:Kailh_socket_MX
- XSW305: renamed from SW305; footprint tamago60:Kailh_socket_MX_platemount -> tamago60:Kailh_socket_MX
- XSW306: renamed from SW306; footprint tamago60:Kailh_socket_MX_platemount -> tamago60:Kailh_socket_MX
- XSW307: renamed from SW307; footprint tamago60:Kailh_socket_MX_platemount -> tamago60:Kailh_socket_MX
- XSW308: renamed from SW308; footprint tamago60:Kailh_socket_MX_platemount -> tamago60:Kailh_socket_MX
- XSW309: renamed from SW309; footprint tamago60:Kailh_socket_MX_platemount -> tamago60:Kailh_socket_MX
- XSW310: renamed from SW310; footprint tamago60:Kailh_socket_MX_platemount -> tamago60:Kailh_socket_MX
- XSW311: renamed from SW311; footprint tamago60:Kailh_socket_MX_platemount -> tamago60:Kailh_socket_MX
- XSW312: renamed from SW312; footprint tamago60:Kailh_socket_MX_platemount -> tamago60:Kailh_socket_MX
- XSW401: renamed from SW401; footprint tamago60:Kailh_socket_MX_platemount -> tamago60:Kailh_socket_MX
- XSW402: renamed from SW402; footprint tamago60:Kailh_socket_MX_platemount -> tamago60:Kailh_socket_MX
- XSW403: renamed from SW403; footprint tamago60:Kailh_socket_MX_platemount -> tamago60:Kailh_socket_MX
- XSW404: renamed from SW404; footprint tamago60:Kailh_socket_MX_platemount -> tamago60:Kailh_socket_MX
- XSW405: renamed from SW405; footprint tamago60:Kailh_socket_MX_platemount -> tamago60:Kailh_socket_MX
- XSW406: renamed from SW406; footprint tamago60:Kailh_socket_MX_platemount -> tamago60:Kailh_socket_MX
- XSW407: renamed from SW407; footprint tamago60:Kailh_socket_MX_platemount -> tamago60:Kailh_socket_MX
- XSW408: renamed from SW408; footprint tamago60:Kailh_socket_MX_platemount -> tamago60:Kailh_socket_MX
- XSW409: renamed from SW409; footprint tamago60:Kailh_socket_MX_platemount -> tamago60:Kailh_socket_MX
- XSW410: renamed from SW410; footprint tamago60:Kailh_socket_MX_platemount -> tamago60:Kailh_socket_MX
- XSW411: renamed from SW411; footprint tamago60:Kailh_socket_MX_platemount -> tamago60:Kailh_socket_MX
- XSW412: renamed from SW412; footprint tamago60:Kailh_socket_MX_platemount -> tamago60:Kailh_socket_MX
- XSW501: renamed from SW501; footprint tamago60:Kailh_socket_MX_platemount -> tamago60:Kailh_socket_MX
- XSW502: renamed from SW502; footprint tamago60:Kailh_socket_MX_platemount -> tamago60:Kailh_socket_MX
- XSW503: renamed from SW503; footprint tamago60:Kailh_socket_MX_platemount -> tamago60:Kailh_socket_MX
- XSW504: renamed from SW504; footprint tamago60:Kailh_socket_MX_platemount -> tamago60:Kailh_socket_MX
- XSW505: renamed from SW505; footprint tamago60:Kailh_socket_MX_platemount -> tamago60:Kailh_socket_MX
- XSW508: renamed from SW508; footprint tamago60:Kailh_socket_MX_platemount -> tamago60:Kailh_socket_MX
- XSW509: renamed from SW509; footprint tamago60:Kailh_socket_MX_platemount -> tamago60:Kailh_socket_MX
- XSW510: renamed from SW510; footprint tamago60:Kailh_socket_MX_platemount -> tamago60:Kailh_socket_MX
- XSW511: renamed from SW511; footprint tamago60:Kailh_socket_MX_platemount -> tamago60:Kailh_socket_MX
- XSW512: renamed from SW512; footprint tamago60:Kailh_socket_MX_platemount -> tamago60:Kailh_socket_MX

Commit message: layout with choc sockets
Parts:
- XSW101, XSW102, XSW103, XSW104, XSW105, XSW106, XSW107, XSW108, XSW109, XSW110, XSW111, XSW112, XSW201, XSW202, XSW203, XSW204, XSW205, XSW206, XSW207, XSW208, XSW209, XSW210, XSW211, XSW212, XSW301, XSW302, XSW303, XSW304, XSW305, XSW306, XSW307, XSW308, XSW309, XSW310, XSW311, XSW312, XSW401, XSW402, XSW403, XSW404, XSW405, XSW406, XSW407, XSW408, XSW409, XSW410, XSW411, XSW412, XSW501, XSW502, XSW503, XSW504, XSW505, XSW508, XSW509, XSW510, XSW511, XSW512: value Kailh MX socket -> Kailh choc socket; footprint tamago60:Kailh_socket_MX -> tamago60:Kailh_socket_PG1350

Commit message: routing
Parts:
- added D506, D507: 1N1418, Diode_SMD:D_SOD-123, symbol Device:D_Small_Filled
- added SW506, SW507: ~, tamago60:SW_D2F-FL, symbol omron_d2f:D2F-FL
Connections:
- net Col6: now also SW506.COM, SW507.COM
- net Row10: now also D507.1 (K)
- net Row5: now also D506.1 (K)
- new net: D506.2 (A), SW506.NO
- new net: D507.2 (A), SW507.NO
- no-connect marks 0 -> 2
Other:
- moved on the sheet: D101, D102, D103, D104, D105, D106, D107, D108, D109, D110, D111, D112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
